Commit message: feat(navigation): freeze validated Nav2 baseline
Chốt cấu hình RPP/NavFn đã chạy trên xe, đồng bộ geometry URDF và footprint, cùng các điều chỉnh bridge/TF trên Pi. Không đổi planner Hz, odom/IMU Hz hay controller sang MPPI trong lần chốt này.

Ghi số liệu goal thẳng và goal phía sau, giới hạn hiện tại và lộ trình A/B tối ưu đường đi/độ mượt sau giai đoạn YOLO. Cập nhật kiểm thử đúng plugin RPP và giữ map quét của người dùng ngoài commit.

File: ros2_ws/src/fire_robot_description/urdf/fire_robot.urdf.xacro (robot description, xacro)
@@ -12,7 +12,7 @@
   <!-- Bánh xe -->
   <xacro:property name="wheel_radius"  value="0.034"/>
-  <xacro:property name="wheel_width"   value="0.026"/>
-  <xacro:property name="track_width"   value="0.180"/>
-  <xacro:property name="wheelbase"     value="0.134"/>
+  <xacro:property name="wheel_width"   value="0.027"/>
+  <xacro:property name="track_width"   value="0.173"/>
+  <xacro:property name="wheelbase"     value="0.135"/>
   <!-- Vị trí cảm biến (Z = ground_clearance + Z_đo_từ_đáy_xe) -->
   <xacro:property name="lidar_x"  value="0.094"/>
